File: kicad_files/MCU.kicad_sch (KiCad schematic)
At the start: 25 parts, among them SW1 Boot, SW2 Reset, U1 RP2040, U2 W25Q128JVS, Y1 12MHz

Commit message: good base
Parts:
- removed SW2: Reset, Button_Switch_SMD:SW_SPST_TL3342, symbol Switch:SW_Push
- SW1: footprint Button_Switch_SMD:SW_SPST_TL3342 -> Connector_PinHeader_2.54mm:PinHeader_1x02_P2.54mm_Vertical
Connections:
- net CAPSLED: no longer names the net of U1.28 (GPIO17)
- net ESCLED: no longer names the net of U1.38 (GPIO26/ADC0)
- net RGBLED: no longer names the net of U1.41 (GPIO29/ADC3)
Other:
- note removed: "Reset Switch"
- title: SST60 - Multi-layout 60% pcb -> Plaket60
Changed lines of the file:
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@@
   (paper "A4")
   (title_block
-    (title "SST60 - Multi-layout 60% pcb")
+    (title "Plaket60")
     (date "2022-07-25")
     (rev "1.0")
@@
     (stroke (width 0) (type default) (color 0 0 0 0))
   )
-  (polyline (pts (xy 163.195 86.36) (xy 196.85 86.36))
-    (stroke (width 0) (type default) (color 0 0 0 0))
-  )
   (wire (pts (xy 49.53 23.495) (xy 52.07 23.495))
     (stroke (width 0) (type default) (color 0 0 0 0))
@@
     (stroke (width 0) (type default) (color 0 0 0 0))
   )
-  (polyline (pts (xy 196.85 86.36) (xy 196.85 107.95))
-    (stroke (width 0) (type default) (color 0 0 0 0))
-  )
   (polyline (pts (xy 95.885 12.7) (xy 95.885 133.35))
     (stroke (width 0) (type default) (color 0 0 0 0))
@@
     (stroke (width 0) (type default) (color 0 0 0 0))
   )
-  (wire (pts (xy 74.93 108.585) (xy 76.835 108.585))
-    (stroke (width 0) (type default) (color 0 0 0 0))
-  )
   (wire (pts (xy 191.77 121.285) (xy 191.77 120.015))
     (stroke (width 0) (type default) (color 0 0 0 0))
@@
   (polyline (pts (xy 95.885 107.95) (xy 163.195 107.95))
     (stroke (width 0) (type default) (color 0 0 0 0))
-  )
-  (text "Reset Switch" (at 163.83 90.17 0)
-    (effects (font (size 1.27 1.27)) (justify left bottom))
   )
   (text "Flash\n" (at 102.235 41.275 180)
@@
     )
   )
-  (global_label "ESCLED" (shape input) (at 74.93 100.965 0) (fields_autoplaced)
-    (effects (font (size 1.27 1.27)) (justify left))
-    (property "Intersheet References" "${INTERSHEET_REFS}" (id 0) (at 84.4188 100.8856 0)
-      (effects (font (size 1.27 1.27)) (justify left) hide)
-    )
-  )
   (global_label "col6" (shape input) (at 76.835 31.115 0) (fields_autoplaced)
     (effects (font (size 1.27 1.27)) (justify left))
@@
     )
   )
-  (global_label "RESET" (shape input) (at 177.165 98.425 180) (fields_autoplaced)
-    (effects (font (size 1.27 1.27)) (justify right))
-    (property "Intersheet References" "${INTERSHEET_REFS}" (id 0) (at 169.0067 98.3456 0)
-      (effects (font (size 1.27 1.27)) (justify right) hide)
-    )
-  )
   (global_label "col3" (shape input) (at 76.835 38.735 0) (fields_autoplaced)
     (effects (font (size 1.27 1.27)) (justify left))
@@
     )
   )
-  (global_label "CAPSLED" (shape input) (at 74.93 74.295 0) (fields_autoplaced)
-    (effects (font (size 1.27 1.27)) (justify left))
-    (property "Intersheet References" "${INTERSHEET_REFS}" (id 0) (at 85.6283 74.2156 0)
-      (effects (font (size 1.27 1.27)) (justify left) hide)
-    )
-  )
   (global_label "RESET" (shape input) (at 25.4 31.115 180) (fields_autoplaced)
     (effects (font (size 1.27 1.27)) (justify right))
@@
     (effects (font (size 1.27 1.27)) (justify left))
     (property "Intersheet References" "${INTERSHEET_REFS}" (id 0) (at 142.7481 28.6544 0)
-      (effects (font (size 1.27 1.27)) (justify left) hide)
-    )
-  )
-  (global_label "RGBLED" (shape input) (at 76.835 108.585 0) (fields_autoplaced)
-    (effects (font (size 1.27 1.27)) (justify left))
-    (property "Intersheet References" "${INTERSHEET_REFS}" (id 0) (at 86.5052 108.5056 0)
       (effects (font (size 1.27 1.27)) (justify left) hide)
     )
@@
     (pin "1")
     (pin "2")
-  )
-  (symbol (lib_id "power:GND") (at 187.325 98.425 0) (unit 1)
-    (in_bom yes) (on_board yes) (fields_autoplaced)
-    (property "Reference" "#PWR0146" (id 0) (at 187.325 104.775 0)
-      (effects (font (size 1.27 1.27)) hide)
-    )
-    (property "Value" "GND" (id 1) (at 187.325 102.87 0))
-    (property "Footprint" "" (id 2) (at 187.325 98.425 0)
-      (effects (font (size 1.27 1.27)) hide)
-    )
-    (property "Datasheet" "" (id 3) (at 187.325 98.425 0)
-      (effects (font (size 1.27 1.27)) hide)
-    )
-    (pin "1")
   )
   (symbol (lib_id "power:GND") (at 191.77 121.285 0) (unit 1)
@@
     (pin "1")
   )
-  (symbol (lib_id "Switch:SW_Push") (at 182.245 98.425 0) (unit 1)
-    (in_bom yes) (on_board yes) (fields_autoplaced)
-    (property "Reference" "SW2" (id 0) (at 182.245 90.17 0))
-    (property "Value" "Reset" (id 1) (at 182.245 92.71 0))
-    (property "Footprint" "Button_Switch_SMD:SW_SPST_TL3342" (id 2) (at 182.245 93.345 0)
-      (effects (font (size 1.27 1.27)) hide)
-    )
-    (property "Datasheet" "~" (id 3) (at 182.245 93.345 0)
-      (effects (font (size 1.27 1.27)) hide)
-    )
-    (pin "1")
-    (pin "2")
-  )
   (symbol (lib_id "power:+3V3") (at 31.75 76.835 0) (unit 1)
     (in_bom yes) (on_board yes)
@@
     (property "Reference" "SW1" (id 0) (at 106.68 50.165 0))
     (property "Value" "Boot" (id 1) (at 106.68 52.705 0))
-    (property "Footprint" "Button_Switch_SMD:SW_SPST_TL3342" (id 2) (at 106.68 52.705 0)
-      (effects (font (size 1.27 1.27)) hide)
-    )
+    (property "Footprint" "Connector_PinHeader_2.54mm:PinHeader_1x02_P2.54mm_Vertical" (id 2) (at 106.68 52.705 0)
+      (effects (font (size 1.27 1.27)) hide)
+    )

Commit message: double jst
Connections:
- net col0: now also U1.28 (GPIO17); no longer U1.32 (GPIO21)
- net row2: now also U1.27 (GPIO16); no longer U1.31 (GPIO20)
- net SCK: now reaches U1.34 (GPIO22)
- new net MATRIX_CS: U1.32 (GPIO21)
- new net MISO: U1.31 (GPIO20)
