File: kicad_files/Misc.kicad_sch (KiCad schematic)
At the start: 19 parts, among them J2 SWD, U5 74AHCT1G125

Commit message: good base
Other:
- title: SST60 - Multi-layout 60% pcb -> Plaket60
Changed lines of the file:
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@@
   (paper "A4")
   (title_block
-    (title "SST60 - Multi-layout 60% pcb")
+    (title "Plaket60")
     (date "2022-07-25")
     (rev "1.0")
