File: kicad_files/Swtich Matrix.kicad_sch (KiCad schematic)
At the start: 147 parts

Commit message: :shower:
Other:
- title: SST60 - Multi-layout 60% pcb -> Plaket60-OG
Changed lines of the file:
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@@
   (paper "A4")
   (title_block
-    (title "SST60 - Multi-layout 60% pcb")
+    (title "Plaket60-OG")
     (date "2022-07-25")
     (rev "1.0")
