File: kicad_files/Swtich Matrix.kicad_sch (KiCad schematic)
At the start: 147 parts

Commit message: good base
Parts:
- removed D24, D29, D47, D52: D_Small, Diode_SMD:D_SOD-123, symbol Device:D_Small
- removed MX1: MX-LED, MX_Alps_Hybrid:MX-1.25U-FLIPPED, symbol cipulot_parts:MX-LED
- removed MX26, MX41, MX57: MX-NoLED, MX_Alps_Hybrid:MX-1U-NoLED, symbol cipulot_parts:MX-NoLED
- removed MX3: MX-LED, MX_Alps_Hybrid:MX-1U, symbol cipulot_parts:MX-LED
- removed MX31: MX-NoLED, MX_Alps_Hybrid:MX-2.25U-ReversedStabilizers-NoLED, symbol cipulot_parts:MX-NoLED
- removed MX32, MX52: MX-NoLED, MX_Alps_Hybrid:MX-3U-ReversedStabilizers-NoLED, symbol cipulot_parts:MX-NoLED
- removed MX5: MX-LED, MX_Alps_Hybrid:MX-1.75U, symbol cipulot_parts:MX-LED
- removed MX51: MX-NoLED, MX_Alps_Hybrid:MX-2.75U-ReversedStabilizers-NoLED, symbol cipulot_parts:MX-NoLED
- removed MX77: MX-NoLED, MX_Alps_Hybrid:MX-10U-ReversedStabilizers-NoLED, symbol cipulot_parts:MX-NoLED
- removed R_LED1, R_LED2: 220, Resistor_SMD:R_0402_1005Metric, symbol Device:R_Small
- added MX3: MX-NoLED, parts:mx_1u, symbol cipulot_parts:MX-NoLED
- added MX5: MX-NoLED, parts:mx_stepped_caps, symbol cipulot_parts:MX-NoLED
- MX10, MX11, MX12, MX13, MX14, MX15, MX16, MX18, MX19, MX20, MX21, MX22, MX23, MX24, MX25, MX27, MX28, MX29, MX30, MX33, MX34, MX35, MX36, MX37, MX38, MX39, MX40, MX43, MX44, MX45, MX46, MX47, MX48, MX49, MX50, MX53, MX54, MX55, MX56, MX58, MX59, MX60, MX61, MX63, MX64, MX65, MX67, MX69, MX73, MX75, MX8, MX9: footprint MX_Alps_Hybrid:MX-1U-NoLED -> parts:mx_1u
- MX17, MX4, MX62, MX7, MX74, MX76: footprint MX_Alps_Hybrid:MX-1.5U-NoLED -> parts:mx_15u
- MX2: footprint MX_Alps_Hybrid:MX-1.25U-NoLED -> parts:mx_125u
- MX42: footprint MX_Alps_Hybrid:MX-7U-ReversedStabilizers-NoLED -> parts:mx_7u
- MX6, MX70: footprint MX_Alps_Hybrid:MX-2.25U-NoLED -> parts:mx_225u
- MX66: footprint MX_Alps_Hybrid:MX-1.75U-NoLED -> parts:mx_175u
- MX68: footprint MX_Alps_Hybrid:MX-2.75U-NoLED -> parts:mx_275u
- MX71: footprint MX_Alps_Hybrid:MX-ISO-ReversedStabilizers -> parts:mx_iso
- MX72: footprint MX_Alps_Hybrid:MX-2U-NoLED -> parts:mx_2u
Connections:
- net col0: now also MX3.1 (COL), MX5.1 (COL)
- net at D1.2 (A): now also MX3.2 (ROW)
- net at D3.2 (A): now also MX5.2 (ROW)
Other:
- title: SST60 - Multi-layout 60% pcb -> Plaket60
- moved on the sheet: D1, D10, D11, D12, D13, D14, D15, D16, D17, D18, D19, D2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
