File: kicad_files/plaket60.kicad_pcb (KiCad board)
At the start: 2 copper layers, 284.7 x 94.2 mm, 164 parts, among them J1 SM04B, J2 SWD, SW1 Boot, U1 RP2040, U2 W25Q128JVS, U3 XC6206PxxxMR, U4 PRTR5V0U2X, Y1 12MHz

Commit message: j'sais pas
Parts:
- J1: footprint Connector_JST:JST_SH_SM04B-SRSS-TB_1x04-1MP_P1.00mm_Horizontal -> Connector_Molex:Molex_Pico-EZmate_78171-0004_1x04-1MP_P1.20mm_Vertical
- moved D12 0.95 mm to (82.5, 50.1)
- moved D16 0.95 mm to (101.5, 50.1)
- moved D20 0.95 mm to (120.6, 50.1)
- moved D25 0.95 mm to (139.6, 50.1)
- moved D30 0.95 mm to (158.7, 50.1)
Routing:
- net col12: track 320.8 -> 320.1 mm
- net GND: vias 72 -> 59

Commit message: double jst
Parts:
- added J3: Conn_01x05, Connector_JST:JST_SH_SM05B-SRSS-TB_1x05-1MP_P1.00mm_Horizontal, B.Cu at (295.4, 58.9)
- J1: footprint Connector_Molex:Molex_Pico-EZmate_78171-0004_1x04-1MP_P1.20mm_Vertical -> Connector_JST:JST_SH_SM04B-SRSS-TB_1x04-1MP_P1.00mm_Horizontal
- moved D34 1.00 mm to (177.7, 50.0)
- moved D39 1.00 mm to (196.8, 50.0)
- moved D43 1.00 mm to (215.8, 50.0)
- moved D48 1.00 mm to (234.9, 50.0)
- moved D53 1.00 mm to (253.9, 50.0)
- moved C_3V-Decoup4 0.57 mm to (52.8, 84.2)
Connections:
- U1 pad 27: unconnected-(U1-Pad27) -> row2
- U1 pad 28: unconnected-(U1-Pad28) -> col0
- U1 pad 31: row2 -> MISO
- U1 pad 32: col0 -> MATRIX_CS
- U1 pad 34: unconnected-(U1-Pad34) -> SCK
Routing:
- net MATRIX_CS: track 0.00 -> 279.2 mm, vias 0 -> 2
- net MISO: track 0.00 -> 277.9 mm, vias 0 -> 2
- net SCK: track 0.00 -> 274.8 mm, vias 0 -> 2
- net +3V3: track 110.3 -> 373.2 mm
- net col0: track 106.8 -> 110.1 mm
- net +1V1: track 27.2 -> 28.8 mm
- net row2: track 267.6 -> 266.9 mm
- net SWCLK: track 28.3 -> 27.7 mm
- net SWDIO: track 26.9 -> 26.4 mm
- net unconnected-(U1-GPIO19-Pad30): track 0.00 -> 0.53 mm
- net GND: track 55.1 -> 54.6 mm, vias 59 -> 61

Commit message: /shrug
Parts:
- moved D57 0.95 mm to (258.7, 126.3)
- moved D10 0.95 mm to (73.0, 126.3)
- moved D38 0.95 mm to (177.7, 126.3)
- moved D62 0.95 mm to (282.5, 126.3)
- moved D58 0.95 mm to (273.0, 50.1)
- moved D15 0.95 mm to (96.8, 126.3)
Routing:
- net MATRIX_CS: track 279.2 -> 282.3 mm
- net SCK: track 274.8 -> 277.9 mm
- net MISO: track 277.9 -> 281.0 mm
- net row4: track 311.5 -> 310.7 mm
- net +3V3: track 373.2 -> 373.8 mm
- net GND: vias 61 -> 60
