File: plaket60.kicad_pcb (KiCad board)
At the start: 2 copper layers, 284.7 x 94.2 mm, 156 parts, among them J2 ISP, J3 ai03_ud, K1 KEYSW, K10 KEYSW, K11 KEYSW, K12 KEYSW, K13 KEYSW, K14 KEYSW, K15 KEYSW, K15-1 KEYSW, K16 KEYSW, K17 KEYSW, K18 KEYSW, K19 KEYSW, K2 KEYSW, K20 KEYSW, K21 KEYSW, K22 KEYSW, K23 KEYSW, K24 KEYSW, K25 KEYSW, K26 KEYSW, K27 KEYSW, K28 KEYSW, K29 KEYSW, K3 KEYSW, K31 KEYSW, K31-1 KEYSW, K32 KEYSW, K33 KEYSW, K34 KEYSW, K35 KEYSW, K36 KEYSW, K37 KEYSW, K38 KEYSW, K39 KEYSW, K4 KEYSW, K40 KEYSW, K41 KEYSW, K42 KEYSW, K43 KEYSW, K44 KEYSW, K44-1 KEYSW, K46 KEYSW, K46-1 KEYSW, K47 KEYSW, K48 KEYSW, K49 KEYSW, K5 KEYSW, K50 KEYSW, K51 KEYSW, K52 KEYSW, K53 KEYSW, K54 KEYSW, K55 KEYSW, K56 KEYSW, K57 KEYSW, K58 KEYSW, K58-1 KEYSW, K59 KEYSW, K6 KEYSW, K61 KEYSW, K62 KEYSW, K63 KEYSW, K67 KEYSW, K7 KEYSW, K72 KEYSW, K73 KEYSW, K74 KEYSW, K8 KEYSW, K9 KEYSW, SW1 SW_PUSH, U1 ATmega32U4, U2 USBLC6-2SC6, X1 XTAL_GND

Commit message: last commit on atmega32u4
Parts:
- moved D11 0.32 mm to (192.6, 10.7)
Routing:
- net GND: track 47.4 -> 135.3 mm, vias 17 -> 7
- net Net-(D44-Pad2): track 43.0 -> 56.9 mm
- net col13: track 372.5 -> 378.3 mm
- net VCC: track 136.5 -> 132.5 mm
- net row3: track 275.7 -> 278.6 mm
- net col0: track 138.5 -> 139.5 mm
- net Net-(D31-Pad2): track 49.6 -> 50.6 mm
- net row4: track 292.0 -> 291.0 mm
- net RST: track 60.0 -> 59.2 mm

Commit message: /shrug
Parts:
- removed the G*** at (87.0, 39.3)
- removed H1: B0, footprints:free_pin
- removed H2: B12, footprints:free_pin
- removed J2: ISP, Keeb_components:isp_standard
- removed X1: XTAL_GND, Keeb_components:Resonator_SMD_muRata_CSTNExxV-3Pin-p1.2
- added C10: 100n, Capacitor_SMD:C_0402_1005Metric, B.Cu at (31.5, 37.0)
- added C11: 100n, Capacitor_SMD:C_0402_1005Metric, B.Cu at (25.4, 35.8)
- added C12: 100n, Capacitor_SMD:C_0402_1005Metric, B.Cu at (31.6, 51.6)
- added C13: 100n, Capacitor_SMD:C_0402_1005Metric, B.Cu at (24.4, 43.8)
- added C14: 100n, Capacitor_SMD:C_0402_1005Metric, B.Cu at (26.3, 47.2)
- added C7: 100n, Capacitor_SMD:C_0402_1005Metric, B.Cu at (30.9, 50.8)
- added C8: 100n, Capacitor_SMD:C_0402_1005Metric, B.Cu at (26.0, 38.7)
- added C9: 100n, Capacitor_SMD:C_0402_1005Metric, B.Cu at (35.4, 39.5)
- added J1: Conn_01x04_Female, Connector_PinHeader_2.54mm:PinHeader_1x04_P2.54mm_Vertical, F.Cu at (4.32, 41.9)
- added R3: 10k, Resistor_SMD:R_0402_1005Metric, B.Cu at (24.0, 51.7)
- added R4: 1k, Resistor_SMD:R_0402_1005Metric, B.Cu at (5.21, 54.1)
- added R7: 5.1k, Resistor_SMD:R_0402_1005Metric, B.Cu at (18.8, 17.5)
- added R8: 10k, Resistor_SMD:R_0402_1005Metric, B.Cu at (19.8, 17.5)
- added SW2: SW_Push, Button_Switch_SMD:SW_SPST_TL3342, B.Cu at (10.1, 54.2)
- added U3: GD25Q80CEIGR, other:USON-8-1EP_3x2mm_P0.5mm_EP0.25x1.65mm, B.Cu at (27.7, 36.5)
- added U4: RP2040, other:RP2040-QFN-56, B.Cu at (30.0, 42.8)
- added Y1: Crystal_GND24, Crystal:Crystal_SMD_3225-4Pin_3.2x2.5mm, B.Cu at (34.9, 49.8)
- C1: value 1u -> 1µ; footprint Keeb_components:C_0805 -> Capacitor_SMD:C_0402_1005Metric
- C2, C5: value 0.1u -> 1µ; footprint Keeb_components:C_0805 -> Capacitor_SMD:C_0402_1005Metric
- C3, C4: value 0.1u -> 15p; footprint Keeb_components:C_0805 -> Capacitor_SMD:C_0402_1005Metric
- C6: value 4.7u -> 1µ; footprint Keeb_components:C_0805 -> Capacitor_SMD:C_0402_1005Metric
- R1, R2: value 22 -> 27; footprint Keeb_components:R_0805 -> Resistor_SMD:R_0402_1005Metric
- R5: footprint Keeb_components:R_0805 -> Resistor_SMD:R_0402_1005Metric
- R6: value 10k -> 1k; footprint Keeb_components:R_0805 -> Resistor_SMD:R_0402_1005Metric
- SW1: value SW_PUSH -> SW_Push
- U1: value ATmega32U4 -> XC6210B332MR-G; footprint Keeb_components:ATMEGA32U4 -> Package_TO_SOT_SMD:SOT-23-5
- moved C2 35.2 mm to (12.2, 20.6), turned to 0 degrees
- moved U1 28.8 mm to (13.0, 18.3), turned to 180 degrees
- moved C4 20.5 mm to (36.1, 52.5), turned to 45 degrees
- moved C1 15.7 mm to (14.1, 20.6)
- moved R5 13.2 mm to (26.8, 34.4), turned to -135 degrees
- moved C5 8.42 mm to (23.6, 44.6), turned to -45 degrees
- moved C6 8.18 mm to (24.1, 41.5), turned to -135 degrees
- moved C3 6.22 mm to (37.5, 51.1), turned to -135 degrees
- moved R1 3.83 mm to (22.0, 20.8), turned to 180 degrees
- moved G*** 3.37 mm to (75.9, 37.7)
- moved G*** 2.04 mm to (141.0, 38.0)
- moved R2 1.13 mm to (21.3, 19.4)
- moved R6 0.93 mm to (33.7, 51.9)
- moved F1 0.50 mm to (16.8, 18.4), turned to -90 degrees
Connections:
- C1 pad 1: Net-(C1-Pad1) -> +5V
- C2 pad 1: GND -> +3V3
- C2 pad 2: VCC -> GND
- C3 pad 1: GND -> Net-(C3-Pad1)
- C3 pad 2: VCC -> GND
- C4 pad 1: GND -> Net-(C4-Pad1)
- C4 pad 2: VCC -> GND
- C5 pad 1: GND -> +3V3
- C5 pad 2: VCC -> GND
- C6 pad 1: GND -> +1V1
- C6 pad 2: VCC -> GND
- F1 pad 1: VCC -> +5V
- J3 pad 2: D- -> DM
- J3 pad 3: D+ -> DP
- R1 pad 2: Net-(R1-Pad2) -> D+
- R2 pad 2: Net-(R2-Pad2) -> D-
- R5 pad 1: RST -> QSPI_CS
- R5 pad 2: VCC -> +3V3
- R6 pad 1: GND -> Net-(C4-Pad1)
- SW1 pad 2: RST -> RESET
- U1 pad 1: row4 -> +5V
- U1 pad 2: VCC -> GND
- U1 pad 3: Net-(R2-Pad2) -> +5V
- U1 pad 4: Net-(R1-Pad1) -> unconnected-(U1-Pad4)
- U1 pad 5: GND -> +3V3
- U2 pad 1: D+ -> DP
- U2 pad 3: D- -> DM
- U2 pad 6: Net-(R1-Pad2) -> Net-(R1-Pad1)
Routing:
- net VCC: track 132.5 -> 0.00 mm, vias 10 -> 0
- net +3V3: track 0.00 -> 97.5 mm, vias 0 -> 2
- net RST: track 59.2 -> 0.00 mm, vias 1 -> 0
- net SWCLK: track 0.00 -> 49.2 mm
- net /VBUS_DET: track 0.00 -> 44.1 mm, vias 0 -> 2
- net QSPI_CS: track 0.00 -> 43.9 mm, vias 0 -> 2
- net SWD: track 0.00 -> 43.8 mm
- net GND: track 135.3 -> 94.3 mm, vias 7 -> 14
- net row1: track 291.1 -> 259.8 mm
- net Net-(R2-Pad2): track 30.2 -> 0.00 mm, vias 2 -> 0
- net Net-(H2-Pad1): track 29.1 -> 0.00 mm
- net Net-(H1-Pad1): track 26.5 -> 0.00 mm
- net col14: track 315.3 -> 290.7 mm
- net MOSI: track 24.0 -> 0.00 mm
- net Net-(R1-Pad1): track 28.6 -> 5.21 mm, vias 2 -> 0
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- added copper zone on B.Cu, net +3V3
Other:
- board text removed: "based on Plain60 Flex Edition by evid13"
