File: plaket60.kicad_sch (KiCad schematic)
At the start: 152 parts, among them J2 ISP, J3 ai03_ud, K1 KEYSW, K10 KEYSW, K11 KEYSW, K12 KEYSW, K13 KEYSW, K14 KEYSW, K15 KEYSW, K15-1 KEYSW, K16 KEYSW, K17 KEYSW, K18 KEYSW, K19 KEYSW, K2 KEYSW, K20 KEYSW, K21 KEYSW, K22 KEYSW, K23 KEYSW, K24 KEYSW, K25 KEYSW, K26 KEYSW, K27 KEYSW, K28 KEYSW, K29 KEYSW, K3 KEYSW, K31 KEYSW, K31-1 KEYSW, K32 KEYSW, K33 KEYSW, K34 KEYSW, K35 KEYSW, K36 KEYSW, K37 KEYSW, K38 KEYSW, K39 KEYSW, K4 KEYSW, K40 KEYSW, K41 KEYSW, K42 KEYSW, K43 KEYSW, K44 KEYSW, K44-1 KEYSW, K46 KEYSW, K46-1 KEYSW, K47 KEYSW, K48 KEYSW, K49 KEYSW, K5 KEYSW, K50 KEYSW, K51 KEYSW, K52 KEYSW, K53 KEYSW, K54 KEYSW, K55 KEYSW, K56 KEYSW, K57 KEYSW, K58 KEYSW, K58-1 KEYSW, K59 KEYSW, K6 KEYSW, K61 KEYSW, K62 KEYSW, K63 KEYSW, K67 KEYSW, K7 KEYSW, K72 KEYSW, K73 KEYSW, K74 KEYSW, K8 KEYSW, K9 KEYSW, SW1 SW_PUSH, U1 ATmega32U4, U2 USBLC6-2SC6, X1 XTAL_GND

Commit message: /shrug
Parts:
- removed H1: B0, footprints:free_pin, symbol Connector_Generic:Conn_01x01
- removed H2: B12, footprints:free_pin, symbol Connector_Generic:Conn_01x01
- removed J2: ISP, Keeb_components:isp_standard, symbol Connector_Generic:Conn_02x03_Odd_Even
- removed SW1: SW_PUSH, Button_Switch_SMD:SW_SPST_TL3342, symbol keyboard_parts:SW_PUSH
- removed U1: ATmega32U4, Keeb_components:ATMEGA32U4, symbol atmel:ATmega32U4
- removed X1: XTAL_GND, Keeb_components:Resonator_SMD_muRata_CSTNExxV-3Pin-p1.2, symbol keyboard_parts:XTAL_GND
- added C10, C11, C12, C13, C14, C7, C8, C9: 100n, Capacitor_SMD:C_0402_1005Metric, symbol Device:C
- added J1: Conn_01x04_Female, Connector_PinHeader_2.54mm:PinHeader_1x04_P2.54mm_Vertical, symbol Connector:Conn_01x04_Female
- added R3, R8: 10k, Resistor_SMD:R_0402_1005Metric, symbol Device:R
- added R4: 1k, Resistor_SMD:R_0402_1005Metric, symbol Device:R
- added R7: 5.1k, Resistor_SMD:R_0402_1005Metric, symbol Device:R
- added SW1, SW2: SW_Push, Button_Switch_SMD:SW_SPST_TL3342, symbol Switch:SW_Push
- added U1: XC6210B332MR-G, Package_TO_SOT_SMD:SOT-23-5, symbol Regulator_Linear:AP2127K-3.3
- added U3: GD25Q80CEIGR, other:USON-8-1EP_3x2mm_P0.5mm_EP0.25x1.65mm, symbol Memory_Flash:W25Q32JVZP
- added U4: RP2040, other:RP2040-QFN-56, symbol MCU_RaspberryPi_RP2040:RP2040
- added Y1: Crystal_GND24, Crystal:Crystal_SMD_3225-4Pin_3.2x2.5mm, symbol Device:Crystal_GND24
- C1: value 1u -> 1µ; footprint Keeb_components:C_0805 -> Capacitor_SMD:C_0402_1005Metric; LCSC (none) -> C19666
- C2: value 0.1u -> 1µ; footprint Keeb_components:C_0805 -> Capacitor_SMD:C_0402_1005Metric; LCSC (none) -> C19666
- C3, C4: value 0.1u -> 15p; footprint Keeb_components:C_0805 -> Capacitor_SMD:C_0402_1005Metric; LCSC (none) -> C1548
- C5: value 0.1u -> 1µ; footprint Keeb_components:C_0805 -> Capacitor_SMD:C_0402_1005Metric; LCSC (none) -> C52923
- C6: value 4.7u -> 1µ; footprint Keeb_components:C_0805 -> Capacitor_SMD:C_0402_1005Metric; LCSC (none) -> C52923
- R1, R2: value 22 -> 27; footprint Keeb_components:R_0805 -> Resistor_SMD:R_0402_1005Metric; LCSC (none) -> C25100
- R5: footprint Keeb_components:R_0805 -> Resistor_SMD:R_0402_1005Metric; LCSC (none) -> C25744
- R6: value 10k -> 1k; footprint Keeb_components:R_0805 -> Resistor_SMD:R_0402_1005Metric; LCSC (none) -> C11702
Connections:
- net D+: now also R1.2, U4.47 (USB_DP); no longer J3.3 (Pin_3), U2.1 (I/O1)
- net D-: now also R2.2, U4.46 (USB_DM); no longer J3.2 (Pin_2), U2.3 (I/O2)
- net GND: now also C2.2, C3.2, C4.2, C5.2, C6.2, C10.2, C11.2, C12.2, C13.2, C14.2, C7.2, C8.2, C9.2, J1.1 (Pin_1), R8.1, SW1.1, SW2.1, U1.2 (GND), U3.4 (GND), U3.9 (EP), U4.19 (TESTEN), U4.57 (GND), Y1.2, Y1.4; no longer C2.1, C3.1, C4.1, C5.1, C6.1, R6.1
- net VBUS: now also R7.2
- net col0: now also U4.41 (GPIO29_ADC3)
- net col1: now also U4.2 (GPIO0)
- net col10: now also U4.8 (GPIO6)
- net col11: now also U4.7 (GPIO5)
- net col12: now also U4.6 (GPIO4)
- net col13: now also U4.5 (GPIO3)
- net col14: now also U4.4 (GPIO2)
- net col2: now also U4.17 (GPIO14)
- net col3: now also U4.16 (GPIO13)
- net col4: now also U4.15 (GPIO12)
- net col5: now also U4.14 (GPIO11)
- net col6: now also U4.13 (GPIO10)
- net col7: now also U4.12 (GPIO9)
- net col8: now also U4.11 (GPIO8)
- net col9: now also U4.9 (GPIO7)
- net row0: now also U4.40 (GPIO28_ADC2)
- net row1: now also U4.3 (GPIO1)
- net row2: now also U4.18 (GPIO15)
- net row3: now also U4.38 (GPIO26_ADC0)
- net row4: now also U4.39 (GPIO27_ADC1)
- net at R6.2: now also U4.21 (XOUT)
- net at R1.1: now also U2.6 (I/O1)
- net +5V: now reaches C1.1
- net +5V: now also F1.1, U1.1 (VIN), U1.3 (EN)
- net RST renamed QSPI_CS
- net QSPI_CS: now also R4.2, U3.1 (~{CS}), U4.56 (QSPI_SS)
- removed net VCC: C2.2, C3.2, C4.2, C5.2, C6.2, F1.1, R5.2
- new net: C3.1, U4.20 (XIN), Y1.1
- new net: C4.1, R6.1, Y1.3
- new net: R4.1, SW2.2
- new net +1V1: C6.1, C7.1, C8.1, U4.23 (DVDD), U4.45 (VREG_VOUT), U4.50 (DVDD)
- new net +3V3: C10.1, C11.1, C12.1, C13.1, C14.1, C2.1, C5.1, C9.1, J1.4 (Pin_4), R3.2, R5.2, U1.5 (VOUT), U3.8 (VCC), U4.1 (IOVDD), U4.10 (IOVDD), U4.22 (IOVDD), U4.33 (IOVDD), U4.42 (IOVDD), U4.43 (ADC_AVDD), U4.44 (VREG_IN), U4.48 (USB_VDD), U4.49 (IOVDD)
- new net DM: J3.2 (Pin_2), U2.3 (I/O2)
- new net DP: J3.3 (Pin_3), U2.1 (I/O1)
- new net QSPI_D0: U3.5 (DI(IO0)), U4.53 (QSPI_SD0)
- new net QSPI_D1: U3.2 (DO(IO1)), U4.55 (QSPI_SD1)
- new net QSPI_D2: U3.3 (IO2), U4.54 (QSPI_SD2)
- new net QSPI_D3: U3.7 (IO3), U4.51 (QSPI_SD3)
- new net QSPI_SCLK: U3.6 (CLK), U4.52 (QSPI_SCLK)
- new net RESET: R3.1, SW1.2, U4.26 (RUN)
- new net SWCLK: J1.3 (Pin_3), U4.24 (SWCLK)
- new net SWD: J1.2 (Pin_2), U4.25 (SWD)
- new net VBUS_DET: R7.1, R8.2, U4.30 (GPIO19)
- no-connect marks 1 -> 9
Other:
- note added: "Buttons"
- note added: "Debug breakout"
- note added: "Decoupling"
- note added: "Flash memory"
- note added: "Matrix"
- note added: "USB-C connector"
- note added: "Voltage regulation"
